File: IoT-Launch-Kit.sch (KiCad schematic (older format))
At the start: 20 parts, among them P1 CONN_01X09, P2 CONN_01X09, U1 LD1117S33CTR, U2 CH340G, U3 ESP-12E, U4 USB-A-PLUG, X1 12MHz

Commit message: v0.2 of the IoT Launch Kit:  - onboard temperature sensor  - only use the side pins of the ESP12 module  - rearrange pin usage  - slim form factor for fitting into USB slot  - NodeMCU style reset circuit
Parts:
- removed P1, P2: CONN_01X09, Pin_Headers:Pin_Header_Straight_1x09, symbol CONN_01X09
- removed U4: USB-A-PLUG, Connect:USB_A, symbol USB-A-PLUG
- removed X1: 12MHz, Crystals:Crystal_HC49-SD_SMD, symbol CRYSTAL
- added P1, P2: CONN_01X08, Pin_Headers:Pin_Header_Straight_1x08, symbol CONN_01X08
- added P3: USB_A, IoT-Launch-Kit:USB_A, symbol USB_A
- added Q1, Q2: S8050, TO_SOT_Packages_SMD:SOT-23, symbol S8050
- added R10, R8, R9: 10k, Resistors_SMD:R_0603, symbol R-RESCUE-IoT-Launch-Kit
- added SW1: SPST, Buttons_Switches_SMD:SW_SPST_FSMSM, symbol SPST
- added U5: LM75A, Housings_SOIC:SOIC-8_3.9x4.9mm_Pitch1.27mm, symbol LM75A
- added X1: CRYSTAL_SMD, Crystals:crystal_FA238-TSX3225, symbol CRYSTAL_SMD
- C1: value 100uF -> 10uF; footprint Capacitors_Tantalum_SMD:TantalC_SizeD_EIA-7343_Reflow -> Capacitors_SMD:C_0805; symbol C -> C-RESCUE-IoT-Launch-Kit
- C2, C3, C4, C5: symbol C -> C-RESCUE-IoT-Launch-Kit
- R1, R2, R3, R4, R5, R6, R7: symbol R -> R-RESCUE-IoT-Launch-Kit
- U3: value ESP-12E -> ESP-12; footprint IoT-Launch-Kit:ESP-12E -> IoT-Launch-Kit:ESP-12; symbol ESP-12E -> ESP-12
Connections:
- net GPIO10 is gone; now on net GPIO0: U3.12 (GPIO0)
- net GPIO9 is gone; now on net GPIO2: U3.11 (GPIO2)
- net +3V3: now also D1.1 (RC), D1.2 (GC), D1.3 (BC), P1.7 (P7), R10.2, U5.5 (A2), U5.6 (A1), U5.7 (A0), U5.8 (VCC)
- net +5V: now also P2.1 (P1), P3.1 (VCC)
- net ADC: now also P1.2 (P2)
- net DIN: now also U3.15 (RXD0), P2.7 (P7); no longer U3.21 (RXD0)
- net DOUT: now also U3.16 (TXD0), P2.8 (P8); no longer U3.22 (TXD0)
- net GND: now also U3.9 (GND), P1.8 (P8), P3.4 (GND), P3.5 (shield), SW1.1, U5.4 (GND), X1.3 (case); no longer U3.15 (GND)
- net GPIO0: now also P2.4 (P4), Q2.3 (C), U5.1 (SDA); no longer U2.13 (DTR), U3.18 (GPIO0)
- net GPIO12: now also R5.2, P1.5 (P5)
- net GPIO13: now also R7.2, P1.6 (P6)
- net GPIO14: now also R6.2, P1.4 (P4)
- net GPIO15: now also U3.10 (GPIO15), P2.2 (P2); no longer U3.16 (GPIO15)
- net GPIO16: now also P1.3 (P3)
- net GPIO2: now also P2.3 (P3), R10.1, U5.2 (SCL); no longer R7.2, U3.17 (GPIO2)
- net GPIO4: now also U3.13 (GPIO4), P2.5 (P5); no longer R6.2, U3.19 (GPIO4)
- net GPIO5: now also U3.14 (GPIO5), P2.6 (P6); no longer R5.2, U3.20 (GPIO5)
- net RST: now also P1.1 (P1), Q1.3 (C), SW1.2; no longer U2.14 (RTS)
- net at U2.5 (D+): now also P3.3 (D+)
- net at U2.6 (D-): now also P3.2 (D-)
- net at C3.1, U2.7 (XI): now also X1.1
- net at C4.1, U2.8 (XO): now also X1.2
- net at D1.4 (BA): now also R7.1
- net at D1.5 (GA): now also R6.1
- net at D1.6 (RA): now also R5.1
- new net: Q2.2 (B), R9.2
- new net: Q1.2 (B), R8.2
- new net DTR: Q2.1 (E), R8.1, U2.13 (DTR)
- new net RTS: Q1.1 (E), R9.1, U2.14 (RTS)
- no-connect marks 9 -> 6
Other:
- moved on the sheet: C1, C2, C3, C4, C5, D1, R1, R2, R3, R4, R5, R6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
